Commit message: Add files via upload

File: robot_core.xacro (robot description, xacro)
@@ -1,4 +1,5 @@
 <?xml version="1.0"?>
 <robot xmlns:xacro="http://www.ros.org/wiki/xacro" >
+    <xacro:include filename="inertial_macros.xacro" />
     <material name="white">
         <color rgba="1 1 1 1" />
@@ -22,12 +23,21 @@
         <origin xyz="-0.1 0 0"/>
     </joint>
-    <link name="chassis">
-        <visual>
-            <origin xyz="0.15 0 0.075" rpy="0 0 0"/>
-            <geometry>
-                <box size="0.3 0.3 0.15"/>
-            </geometry>
-                <material name="white"/>
-        </visual>
+   <link name="chassis">
+    <visual>
+        <origin xyz="0.15 0 0.075" rpy="0 0 0"/>
+        <geometry>
+            <box size="0.3 0.3 0.15"/>
+        </geometry>
+        <material name="white"/>
+    </visual>
+    <collision>
+        <origin xyz="0.15 0 0.075" rpy="0 0 0"/>
+        <geometry>
+            <box size="0.3 0.3 0.15"/>
+        </geometry>
+    </collision>
+        <xacro:inertial_box mass="0.5" x="0.3" y="0.3" z="0.15">
+         <origin xyz="0.15 0 0.075" rpy="0 0 0"/>
+        </xacro:inertial_box>
     </link>
     <link name="base_link">
@@ -47,4 +57,7 @@
         <material name="blue"/>
     </visual>
+        <xacro:inertial_cylinder mass="0.1" length="0.05" radius="0.05">
+          <origin xyz="0 0 0" rpy="0 0 0"/>
+        </xacro:inertial_cylinder>
     </link>
     <!-- RIGHT WHEEL -->
@@ -62,4 +75,24 @@
         <material name="blue"/>
     </visual>
+        <xacro:inertial_cylinder mass="0.1" length="0.05" radius="0.05">
+          <origin xyz="0 0 0" rpy="0 0 0"/>
+        </xacro:inertial_cylinder>
+    </link>
+    <!-- CASTER WHEEL -->
+    <joint name="caster_wheel_joint" type="fixed">
+    <parent link="chassis"/>
+    <child link="caster_wheel"/>
+    <origin xyz="0.24 0 0" rpy="0 0 0"/>
+    </joint>
+    <link name="caster_wheel">
+    <visual>
+        <geometry>
+            <sphere radius="0.05" />
+        </geometry>
+        <material name="black"/>
+    </visual>
+        <xacro:inertial_cylinder mass="0.1" length="0.05" radius="0.05">
+          <origin xyz="0 0 0" rpy="0 0 0"/>
+        </xacro:inertial_cylinder>
     </link>
 </robot>

Commit message: Add files via upload

File: robot_core.xacro (robot description, xacro)
@@ -23,21 +23,22 @@
         <origin xyz="-0.1 0 0"/>
     </joint>
-   <link name="chassis">
-    <visual>
-        <origin xyz="0.15 0 0.075" rpy="0 0 0"/>
-        <geometry>
-            <box size="0.3 0.3 0.15"/>
-        </geometry>
-        <material name="white"/>
-    </visual>
-    <collision>
-        <origin xyz="0.15 0 0.075" rpy="0 0 0"/>
-        <geometry>
-            <box size="0.3 0.3 0.15"/>
-        </geometry>
-    </collision>
-        <xacro:inertial_box mass="0.5" x="0.3" y="0.3" z="0.15">
-         <origin xyz="0.15 0 0.075" rpy="0 0 0"/>
-        </xacro:inertial_box>
+    <link name="chassis">
+        <visual>
+            <origin xyz="0.15 0 0.075" rpy="0 0 0"/>
+            <geometry>
+                <box size="0.3 0.3 0.15"/>
+            </geometry>
+            <material name="white"/>
+        </visual>
+        <collision>
+            <origin xyz="0.15 0 0.075" rpy="0 0 0"/>
+            <geometry>
+                <box size="0.3 0.3 0.15"/>
+            </geometry>
+        </collision>
+            <!-- ... visual and collision here ... -->
+            <xacro:inertial_box mass="0.5" x="0.3" y="0.3" z="0.15">
+                <origin xyz="0.15 0 0.075" rpy="0 0 0"/>
+            </xacro:inertial_box>
     </link>
     <link name="base_link">
@@ -51,13 +52,14 @@
     </joint>
     <link name="left_wheel">
-    <visual>
-        <geometry>
-            <cylinder length="0.04" radius="0.05" />
-        </geometry>
-        <material name="blue"/>
-    </visual>
-        <xacro:inertial_cylinder mass="0.1" length="0.05" radius="0.05">
-          <origin xyz="0 0 0" rpy="0 0 0"/>
-        </xacro:inertial_cylinder>
+        <visual>
+            <geometry>
+                <cylinder length="0.04" radius="0.05" />
+            </geometry>
+            <material name="blue"/>
+        </visual>
+            <!-- ... visual and collision here ... -->
+            <xacro:inertial_cylinder mass="0.1" length="0.05" radius="0.05">
+                <origin xyz="0 0 0" rpy="0 0 0"/>
+            </xacro:inertial_cylinder>
     </link>
     <!-- RIGHT WHEEL -->
@@ -69,30 +71,32 @@
     </joint>
     <link name="right_wheel">
-    <visual>
-        <geometry>
-            <cylinder length="0.04" radius="0.05" />
-        </geometry>
-        <material name="blue"/>
-    </visual>
-        <xacro:inertial_cylinder mass="0.1" length="0.05" radius="0.05">
-          <origin xyz="0 0 0" rpy="0 0 0"/>
-        </xacro:inertial_cylinder>
+        <visual>
+            <geometry>
+                <cylinder length="0.04" radius="0.05" />
+            </geometry>
+            <material name="blue"/>
+        </visual>
+            <!-- ... visual and collision here ... -->
+            <xacro:inertial_cylinder mass="0.1" length="0.05" radius="0.05">
+                <origin xyz="0 0 0" rpy="0 0 0"/>
+            </xacro:inertial_cylinder>
     </link>
     <!-- CASTER WHEEL -->
     <joint name="caster_wheel_joint" type="fixed">
-    <parent link="chassis"/>
-    <child link="caster_wheel"/>
-    <origin xyz="0.24 0 0" rpy="0 0 0"/>
+        <parent link="chassis"/>
+        <child link="caster_wheel"/>
+        <origin xyz="0.24 0 0" rpy="0 0 0"/>
     </joint>
     <link name="caster_wheel">
-    <visual>
-        <geometry>
-            <sphere radius="0.05" />
-        </geometry>
-        <material name="black"/>
-    </visual>
-        <xacro:inertial_cylinder mass="0.1" length="0.05" radius="0.05">
-          <origin xyz="0 0 0" rpy="0 0 0"/>
-        </xacro:inertial_cylinder>
+        <visual>
+            <geometry>
+                <sphere radius="0.05" />
+            </geometry>
+            <material name="black"/>
+        </visual>
+            <!-- ... visual and collision here ... -->
+            <xacro:inertial_sphere mass="0.1" radius="0.05">
+                <origin xyz="0 0 0" rpy="0 0 0"/>
+            </xacro:inertial_sphere>
     </link>
 </robot>
