Commit message: Add files via upload

File: robot.urdf.xacro (robot description, xacro)
@@ -2,3 +2,5 @@
 <robot xmlns:xacro="http://www.ros.org/wiki/xacro"  name="robot">
     <xacro:include filename="robot_core.xacro" />
+    <xacro:include filename="robot_teleop_core.xacro" />
+    <xacro:include filename="gazebo_control.xacro" />
 </robot>

File: robot_core.xacro (robot description, xacro)
@@ -21,23 +21,24 @@
         <parent link="base_link"/>
         <child link="chassis"/>
-        <origin xyz="-0.1 0 0"/>
+        <origin xyz="0 0 0.05"/>
     </joint>
-   <link name="chassis">
-    <visual>
-        <origin xyz="0.15 0 0.075" rpy="0 0 0"/>
-        <geometry>
-            <box size="0.5 0.5 0.15"/>
-        </geometry>
-        <material name="white"/>
-    </visual>
-    <collision>
-        <origin xyz="0.15 0 0.075" rpy="0 0 0"/>
-        <geometry>
-            <box size="0.5 0.5 0.15"/>
-        </geometry>
-    </collision>
-        <xacro:inertial_box mass="0.5" x="0.3" y="0.3" z="0.15">
-         <origin xyz="0.15 0 0.075" rpy="0 0 0"/>
-        </xacro:inertial_box>
+    <link name="chassis">
+        <visual>
+            <origin xyz="0 0 0.05" rpy="0 0 0"/>
+            <geometry>
+                <box size="0.5 0.3 0.2"/>
+            </geometry>
+            <material name="white"/>
+        </visual>
+        <collision>
+            <origin xyz="0 0 0.05" rpy="0 0 0"/>
+            <geometry>
+                <box size="0.5 0.3 0.2"/>
+            </geometry>
+        </collision>
+            <!-- ... visual and collision here ... -->
+            <xacro:inertial_box mass="0.5" x="0.5" y="0.3" z="0.2">
+                <origin xyz="0 0 0.05" rpy="0 0 0"/>
+            </xacro:inertial_box>
     </link>
     <link name="base_link">
@@ -47,71 +48,117 @@
         <parent link="base_link"/>
         <child link="left_front_wheel"/>
-        <origin xyz="0.25 0.25 0" rpy="-${pi/2} 0 0"/>
+        <origin xyz="0.15 -0.1 0" rpy="-${pi/2} 0 0"/>
         <axis xyz="0 0 1"/>
     </joint>
     <link name="left_front_wheel">
-    <visual>
-        <geometry>
-            <cylinder length="0.04" radius="0.05" />
-        </geometry>
-        <material name="blue"/>
-    </visual>
-        <xacro:inertial_cylinder mass="0.1" length="0.04" radius="0.05">
-          <origin xyz="0 0 0" rpy="0 0 0"/>
-        </xacro:inertial_cylinder>
-    </link>
-    <!-- RIGHT FRONT WHEEL -->
-    <joint name="right_wheel_joint" type="continuous">
-        <parent link="base_link"/>
-        <child link="right_wheel"/>
-        <origin xyz="0.25 -0.25 0" rpy="${pi/2} 0 0"/>
-        <axis xyz="0 0 -1"/>
-    </joint>
-    <link name="right_wheel">
-    <visual>
-        <geometry>
-            <cylinder length="0.04" radius="0.05" />
-        </geometry>
-        <material name="red"/>
-    </visual>
-        <xacro:inertial_cylinder mass="0.1" length="0.04" radius="0.05">
-          <origin xyz="0 0 0" rpy="0 0 0"/>
-        </xacro:inertial_cylinder>
+        <visual>
+            <geometry>
+                <cylinder length="0.04" radius="0.05" />
+            </geometry>
+            <material name="orange"/>
+        </visual>
+            <!-- ... visual and collision here ... -->
+            <xacro:inertial_cylinder mass="0.1" length="0.05" radius="0.05">
+                <origin xyz="0 0 0" rpy="0 0 0"/>
+            </xacro:inertial_cylinder>
+        <collision>
+            <origin xyz="0.15 -0.1 0" rpy="-${pi/2} 0 0"/>
+            <geometry>
+                <cylinder length="0.04" radius="0.05" />
+            </geometry>
+        </collision>
     </link>
     <!-- LEFT BACK WHEEL -->
-    <joint name="left_back_wheel_joint" type="continuous">
+    <joint name="left_back_wheel_joint" type="fixed">
         <parent link="base_link"/>
         <child link="left_back_wheel"/>
-        <origin xyz="-0.15 0.25 0" rpy="-${pi/2} 0 0"/>
+        <origin xyz="-0.15 -0.1 0" rpy="-${pi/2} 0 0"/>
         <axis xyz="0 0 1"/>
     </joint>
     <link name="left_back_wheel">
-    <visual>
-        <geometry>
-            <cylinder length="0.04" radius="0.05" />
-        </geometry>
-        <material name="orange"/>
-    </visual>
-        <xacro:inertial_cylinder mass="0.1" length="0.04" radius="0.05">
-          <origin xyz="0 0 0" rpy="0 0 0"/>
-        </xacro:inertial_cylinder>
+        <visual>
+            <geometry>
+                <cylinder length="0.04" radius="0.05" />
+            </geometry>
+            <material name="blue"/>
+        </visual>
+            <!-- ... visual and collision here ... -->
+            <xacro:inertial_cylinder mass="0.1" length="0.05" radius="0.05">
+                <origin xyz="0 0 0" rpy="0 0 0"/>
+            </xacro:inertial_cylinder>
+        <collision>
+            <origin xyz="-0.15 -0.1 0" rpy="-${pi/2} 0 0"/>
+            <geometry>
+                <cylinder length="0.04" radius="0.05" />
+            </geometry>
+        </collision>
+    </link>
+    <!-- RIGHT FRONT WHEEL -->
+    <joint name="right_front_wheel_joint" type="continuous">
+        <parent link="base_link"/>
+        <child link="right_front_wheel"/>
+        <origin xyz="0.15 0.1 0" rpy="${pi/2} 0 0"/>
+        <axis xyz="0 0 -1"/>
+    </joint>
+    <link name="right_front_wheel">
+        <visual>
+            <geometry>
+                <cylinder length="0.04" radius="0.05" />
+            </geometry>
+            <material name="red"/>
+        </visual>
+            <!-- ... visual and collision here ... -->
+            <xacro:inertial_cylinder mass="0.1" length="0.05" radius="0.05">
+                <origin xyz="0 0 0" rpy="0 0 0"/>
+            </xacro:inertial_cylinder>
+         <collision>
+            <origin xyz="0.15 0.1 0" rpy="-${pi/2} 0 0"/>
+            <geometry>
+                <cylinder length="0.04" radius="0.05" />
+            </geometry>
+        </collision>
     </link>
     <!-- RIGHT BACK WHEEL -->
-    <joint name="right_back_wheel_joint" type="continuous">
+    <joint name="right_back_wheel_joint" type="fixed">
         <parent link="base_link"/>
         <child link="right_back_wheel"/>
-        <origin xyz="-0.15 -0.25 0" rpy="${pi/2} 0 0"/>
+        <origin xyz="-0.15 0.1 0" rpy="${pi/2} 0 0"/>
         <axis xyz="0 0 -1"/>
     </joint>
     <link name="right_back_wheel">
+        <visual>
+            <geometry>
+                <cylinder length="0.04" radius="0.05" />
+            </geometry>
+            <material name="black"/>
+        </visual>
+            <!-- ... visual and collision here ... -->
+            <xacro:inertial_cylinder mass="0.1" length="0.05" radius="0.05">
+                <origin xyz="0 0 0" rpy="0 0 0"/>
+            </xacro:inertial_cylinder>
+        <collision>
+            <origin xyz="-0.15 0.1 0" rpy="-${pi/2} 0 0"/>
+            <geometry>
+                <cylinder length="0.04" radius="0.05" />
+            </geometry>
+        </collision>
+    </link>
+    <!-- CASTER WHEEL -->
+    <joint name="caster_wheel_joint" type="fixed">
+        <parent link="chassis"/>
+        <child link="caster_wheel"/>
+        <origin xyz="0.24 0 0" rpy="0 0 0"/>
+    </joint>
+    <link name="caster_wheel">
     <visual>
         <geometry>
-            <cylinder length="0.04" radius="0.05" />
+            <sphere radius="0.05" />
         </geometry>
         <material name="black"/>
     </visual>
-        <xacro:inertial_cylinder mass="0.1" length="0.04" radius="0.05">
-          <origin xyz="0 0 0" rpy="0 0 0"/>
-        </xacro:inertial_cylinder>
+      <!-- ... visual and collision here ... -->
+        <xacro:inertial_sphere mass="0.1" radius="0.05">
+            <origin xyz="0 0 0" rpy="0 0 0"/>
+        </xacro:inertial_sphere>
     </link>
 </robot>
