Commit message: Update robot_core.xacro

File: Lab05/description/robot_core.xacro (robot description, xacro)
@@ -18,38 +18,40 @@
     </material>
     <!-- BASE LINK -->
+    <link name="base_link">
+    </link>
     <joint name="chassis_joint" type="fixed">
         <parent link="base_link"/>
         <child link="chassis"/>
-        <origin xyz="0 0 0.05"/>
+        <origin xyz="-0.1 0 0"/>
     </joint>
     <link name="chassis">
         <visual>
-            <origin xyz="0 0 0.05" rpy="0 0 0"/>
+            <origin xyz="0.15 0 0.075" rpy="0 0 0"/>
             <geometry>
-                <box size="0.5 0.3 0.2"/>
+                <box size="0.3 0.3 0.15"/>
             </geometry>
             <material name="white"/>
         </visual>
         <collision>
-            <origin xyz="0 0 0.05" rpy="0 0 0"/>
+            <origin xyz="0.15 0 0.075" rpy="0 0 0"/>
             <geometry>
-                <box size="0.5 0.3 0.2"/>
+                <box size="0.3 0.3 0.15"/>
             </geometry>
         </collision>
-            <!-- ... visual and collision here ... -->
-            <xacro:inertial_box mass="0.5" x="0.5" y="0.3" z="0.2">
-                <origin xyz="0 0 0.05" rpy="0 0 0"/>
-            </xacro:inertial_box>
+        <xacro:inertial_box mass="0.5" x="0.3" y="0.3" z="0.15">
+            <origin xyz="0.15 0 0.075" rpy="0 0 0"/>
+        </xacro:inertial_box>
     </link>
-    <link name="base_link">
-    </link>
-    <!-- LEFT FRONT WHEEL -->
-    <joint name="left_front_wheel_joint" type="continuous">
+    <gazebo reference="chassis">
+        <material>Gazebo/White</material>
+    </gazebo>
+    <!-- LEFT WHEEL -->
+    <joint name="left_wheel_joint" type="continuous">
         <parent link="base_link"/>
-        <child link="left_front_wheel"/>
-        <origin xyz="0.15 -0.1 0" rpy="-${pi/2} 0 0"/>
+        <child link="left_wheel"/>
+        <origin xyz="0 0.175 0" rpy="-${pi/2} 0 0"/>
         <axis xyz="0 0 1"/>
     </joint>
-    <link name="left_front_wheel">
+    <link name="left_wheel">
         <visual>
             <geometry>
@@ -58,48 +60,24 @@
             <material name="orange"/>
         </visual>
-            <!-- ... visual and collision here ... -->
-            <xacro:inertial_cylinder mass="0.1" length="0.05" radius="0.05">
-                <origin xyz="0 0 0" rpy="0 0 0"/>
-            </xacro:inertial_cylinder>
         <collision>
-            <origin xyz="0.15 -0.1 0" rpy="-${pi/2} 0 0"/>
             <geometry>
                 <cylinder length="0.04" radius="0.05" />
             </geometry>
         </collision>
+        <xacro:inertial_cylinder mass="0.1" length="0.05" radius="0.05">
+            <origin xyz="0 0 0" rpy="0 0 0"/>
+        </xacro:inertial_cylinder>
     </link>
-    <!-- LEFT BACK WHEEL -->
-    <joint name="left_back_wheel_joint" type="fixed">
+    <gazebo reference="left_wheel">
+        <material>Gazebo/Orange</material>
+    </gazebo>
+    <!-- RIGHT WHEEL -->
+    <joint name="right_wheel_joint" type="continuous">
         <parent link="base_link"/>
-        <child link="left_back_wheel"/>
-        <origin xyz="-0.15 -0.1 0" rpy="-${pi/2} 0 0"/>
-        <axis xyz="0 0 1"/>
-    </joint>
-    <link name="left_back_wheel">
-        <visual>
-            <geometry>
-                <cylinder length="0.04" radius="0.05" />
-            </geometry>
-            <material name="blue"/>
-        </visual>
-            <!-- ... visual and collision here ... -->
-            <xacro:inertial_cylinder mass="0.1" length="0.05" radius="0.05">
-                <origin xyz="0 0 0" rpy="0 0 0"/>
-            </xacro:inertial_cylinder>
-        <collision>
-            <origin xyz="-0.15 -0.1 0" rpy="-${pi/2} 0 0"/>
-            <geometry>
-                <cylinder length="0.04" radius="0.05" />
-            </geometry>
-        </collision>
-    </link>
-    <!-- RIGHT FRONT WHEEL -->
-    <joint name="right_front_wheel_joint" type="continuous">
-        <parent link="base_link"/>
-        <child link="right_front_wheel"/>
-        <origin xyz="0.15 0.1 0" rpy="${pi/2} 0 0"/>
+        <child link="right_wheel"/>
+        <origin xyz="0 -0.175 0" rpy="${pi/2} 0 0"/>
         <axis xyz="0 0 -1"/>
     </joint>
-    <link name="right_front_wheel">
+    <link name="right_wheel">
         <visual>
             <geometry>
@@ -108,40 +86,16 @@
             <material name="red"/>
         </visual>
-            <!-- ... visual and collision here ... -->
-            <xacro:inertial_cylinder mass="0.1" length="0.05" radius="0.05">
-                <origin xyz="0 0 0" rpy="0 0 0"/>
-            </xacro:inertial_cylinder>
-         <collision>
-            <origin xyz="0.15 0.1 0" rpy="-${pi/2} 0 0"/>
+        <collision>
             <geometry>
                 <cylinder length="0.04" radius="0.05" />
             </geometry>
         </collision>
+        <xacro:inertial_cylinder mass="0.1" length="0.05" radius="0.05">
+            <origin xyz="0 0 0" rpy="0 0 0"/>
+        </xacro:inertial_cylinder>
     </link>
-    <!-- RIGHT BACK WHEEL -->
-    <joint name="right_back_wheel_joint" type="fixed">
-        <parent link="base_link"/>
-        <child link="right_back_wheel"/>
-        <origin xyz="-0.15 0.1 0" rpy="${pi/2} 0 0"/>
-        <axis xyz="0 0 -1"/>
-    </joint>
-    <link name="right_back_wheel">
-        <visual>
-            <geometry>
-                <cylinder length="0.04" radius="0.05" />
-            </geometry>
-            <material name="black"/>
-        </visual>
-            <!-- ... visual and collision here ... -->
-            <xacro:inertial_cylinder mass="0.1" length="0.05" radius="0.05">
-                <origin xyz="0 0 0" rpy="0 0 0"/>
-            </xacro:inertial_cylinder>
-        <collision>
-            <origin xyz="-0.15 0.1 0" rpy="-${pi/2} 0 0"/>
-            <geometry>
-                <cylinder length="0.04" radius="0.05" />
-            </geometry>
-        </collision>
-    </link>
+    <gazebo reference="right_wheel">
+        <material>Gazebo/Red</material>
+    </gazebo>
     <!-- CASTER WHEEL -->
     <joint name="caster_wheel_joint" type="fixed">
@@ -151,14 +105,23 @@
     </joint>
     <link name="caster_wheel">
-    <visual>
-        <geometry>
-            <sphere radius="0.05" />
-        </geometry>
-        <material name="black"/>
-    </visual>
-      <!-- ... visual and collision here ... -->
+        <visual>
+            <geometry>
+                <sphere radius="0.05" />
+            </geometry>
+            <material name="blue"/>
+        </visual>
+        <collision>
+            <geometry>
+                <sphere radius="0.05" />
+            </geometry>
+        </collision>
         <xacro:inertial_sphere mass="0.1" radius="0.05">
             <origin xyz="0 0 0" rpy="0 0 0"/>
         </xacro:inertial_sphere>
     </link>
+    <gazebo reference="caster_wheel">
+        <material>Gazebo/Blue</material>
+        <mu1 value="0"/>
+        <mu2 value="0"/>
+    </gazebo>
 </robot>
